File: Video-Ball.kicad_pcb (KiCad board)
At the start: 2 copper layers, 225.7 x 123.5 mm, 21 parts, among them U1 74HC00, U10 74HC00, U11 74HC00, U12 74HC00, U13 74HC00, U2 74HC00, U3 74HC00, U4 74HC02, U5 74HC00, U6 74HC00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

Commit message: Fixed incorrect silk screen said HR and D under IC U1 should be a 330pF cap
Other:
- board text removed: "H R"
Changed lines of the file:
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@@
   (gr_rect (start 172.37 76.44) (end 165.83 73.7) (layer "F.SilkS") (width 0.15) (fill none))
   (gr_arc (start 95.75 106.6) (mid 96.457107 106.892893) (end 96.75 107.6) (layer "F.SilkS") (width 0.15))
+  (gr_arc (start 96.75 67.603553) (mid 97.457096 67.896457) (end 97.75 68.603553) (layer "F.SilkS") (width 0.15))
   (gr_line (start 112.05 36.5) (end 112.95 36.5) (layer "F.SilkS") (width 0.15))
   (gr_line (start 83.54 39.87) (end 85.07 39.87) (layer "F.SilkS") (width 0.15))
@@
   (gr_line (start 143.5 45.1) (end 143.5 42.307107) (layer "F.SilkS") (width 0.15))
   (gr_line (start 81 77.1) (end 81 74.307107) (layer "F.SilkS") (width 0.15))
+  (gr_line (start 97.75 68.603553) (end 97.75 71.396446) (layer "F.SilkS") (width 0.15))
   (gr_rect (start 153.6 132.74) (end 155.84 128.5) (layer "F.SilkS") (width 0.15) (fill none))
   (gr_arc (start 187 95.407107) (mid 187.707104 95.700001) (end 188 96.407107) (layer "F.SilkS") (width 0.15))
@@
   (gr_line (start 109.8 52.05) (end 112.65 52.05) (layer "F.SilkS") (width 0.15))
   (gr_line (start 83.67 35.43) (end 85.2 35.43) (layer "F.SilkS") (width 0.15))
+  (gr_arc (start 96.75 72.396446) (mid 96.042904 72.103542) (end 95.75 71.396446) (layer "F.SilkS") (width 0.15))
   (gr_line (start 53.8 110.48) (end 45.2 110.46) (layer "F.SilkS") (width 0.15))
   (gr_line (start 61.97 93.53) (end 63.5 93.53) (layer "F.SilkS") (width 0.15))
@@
   (gr_rect (start 83.54 41.24) (end 77 38.5) (layer "F.SilkS") (width 0.15) (fill none))
   (gr_rect (start 120.4 57.93) (end 117.66 64.47) (layer "F.SilkS") (width 0.15) (fill none))
+  (gr_arc (start 97.75 71.396446) (mid 97.457113 72.103559) (end 96.75 72.396446) (layer "F.SilkS") (width 0.15))
   (gr_line (start 108.45 108.5) (end 108.4 131.2) (layer "F.SilkS") (width 0.3))
   (gr_arc (start 91.75 54.6) (mid 91.457107 55.307107) (end 90.75 55.6) (layer "F.SilkS") (width 0.15))
@@
   (gr_rect (start 188.24 80.53) (end 185.5 87.07) (layer "F.SilkS") (width 0.15) (fill none))
   (gr_rect (start 198.04 139.6) (end 191.5 136.86) (layer "F.SilkS") (width 0.15) (fill none))
+  (gr_line (start 95.75 71.396446) (end 95.75 68.603553) (layer "F.SilkS") (width 0.15))
   (gr_line (start 111.15 38.1) (end 111.15 39.55) (layer "F.SilkS") (width 0.15))
   (gr_arc (start 98 96.6) (mid 97.707107 97.307107) (end 97 97.6) (layer "F.SilkS") (width 0.15))
@@
   (gr_line (start 193.6 85.6) (end 193.6 82.807107) (layer "F.SilkS") (width 0.15))
   (gr_arc (start 201 65.807107) (mid 201.292891 65.099996) (end 202 64.807107) (layer "F.SilkS") (width 0.15))
-  (gr_line (start 154.72 132.74) (end 154.72 138.1) (layer "F.SilkS") (width 0.15))
+  (gr_line (start 154.72 132.74) (end 154.72 134.4) (layer "F.SilkS") (width 0.15))
   (gr_arc (start 170 58.1) (mid 169.707107 58.807107) (end 169 59.1) (layer "F.SilkS") (width 0.15))
   (gr_line (start 173.25 104.2) (end 176.042893 104.2) (layer "F.SilkS") (width 0.15))
@@
   (gr_line (start 131.77 112.17) (end 131.77 113.8) (layer "F.SilkS") (width 0.15))
   (gr_arc (start 123 112.807107) (mid 123.292891 112.099996) (end 124 111.807107) (layer "F.SilkS") (width 0.15))
+  (gr_line (start 96.75 72.448224) (end 96.75 74) (layer "F.SilkS") (width 0.3))
   (gr_line (start 75 102.307107) (end 75 98.85) (layer "F.SilkS") (width 0.15))
   (gr_line (start 125 112.807107) (end 125 115.6) (layer "F.SilkS") (width 0.15))
@@
   (gr_arc (start 150.5 46.1) (mid 149.792893 45.807107) (end 149.5 45.1) (layer "F.SilkS") (width 0.15))
   (gr_rect (start 46.64 86.64) (end 46.4 84.4) (layer "F.SilkS") (width 0.15) (fill solid))
+  (gr_line (start 96.75 66.448224) (end 96.75 67.551777) (layer "F.SilkS") (width 0.3))
   (gr_rect (start 90.17 134.3) (end 83.63 131.56) (layer "F.SilkS") (width 0.15) (fill none))
   (gr_line (start 113.88 112.72) (end 113.88 119.6) (layer "F.SilkS") (width 0.15))
@@
   (gr_circle (center 246.8 63.798685) (end 246.9 59.998685) (layer "F.SilkS") (width 0.15) (fill none))
   (gr_line (start 105.3 110.4) (end 105.45 124.9) (layer "F.SilkS") (width 0.3))
+  (gr_arc (start 95.75 68.603553) (mid 96.042895 67.896447) (end 96.75 67.603553) (layer "F.SilkS") (width 0.15))
   (gr_rect (start 178.26 128.04) (end 180.5 127.8) (layer "F.SilkS") (width 0.15) (fill solid))
   (gr_arc (start 92.957107 108.6) (mid 92.249996 108.307109) (end 91.957107 107.6) (layer "F.SilkS") (width 0.15))
@@
     (effects (font (size 1 1) (thickness 0.15)))
   )
-  (gr_text "H R\n" (at 99.8 75.4 90) (layer "F.SilkS")
-    (effects (font (size 1 1) (thickness 0.15)))
-  )
   (gr_text "470k" (at 126.6 41.2) (layer "F.SilkS")
     (effects (font (size 1 1) (thickness 0.15)))
@@
     (effects (font (size 1 1) (thickness 0.15)))
   )
-  (gr_text "D" (at 96.8 62.6 90) (layer "F.SilkS")
-    (effects (font (size 1 1) (thickness 0.15)))
-  )
   (gr_text "2200μ" (at 236.6 49.410874 90) (layer "F.SilkS")
     (effects (font (size 1 1) (thickness 0.15)))
@@
   )
   (gr_text "10n" (at 97 95.1 90) (layer "F.SilkS")
+    (effects (font (size 1 1) (thickness 0.15)))
+  )
+  (gr_text "330p\n" (at 96.75 70 90) (layer "F.SilkS")
     (effects (font (size 1 1) (thickness 0.15)))
   )
@@
     (effects (font (size 1 1) (thickness 0.15)))
   )
-  (gr_text "33n" (at 156.5 81.6) (layer "F.SilkS")
+  (gr_text "33n\n" (at 156.5 81.6) (layer "F.SilkS")
     (effects (font (size 1 1) (thickness 0.15)))
   )
@@
     (effects (font (size 1 1) (thickness 0.15)))
   )
-  (gr_text "+" (at 242.1 37.4 90) (layer "F.SilkS")
+  (gr_text "+" (at 242.5 37.4 90) (layer "F.SilkS")
     (effects (font (size 2 2) (thickness 0.15)))
   )
@@
     )
   )
+  (group "" (id 12386862-ab1d-4ef9-8db8-21da0effcd15)
+    (members
+      1c4d3570-b802-461a-8af2-927a3a5cc8c4
+      2ca97b87-01ea-47c9-96b4-83317d16b26c
+      3b02c02a-9ad1-4a5d-a004-416ac74a8b10
+      440ab49c-58b9-43f5-bcf8-7ef6a7b96f3f
+      6980f22c-329e-47fc-a086-f14814c3f92b
+      cd7c450e-ed9d-4411-a6de-2e5fcfffda70
+    )
+  )
